Commit message: URDF functionality complete

File: flo_URDF.urdf (robot description, URDF)
Before this commit: robot Lil_Flo, 17 links, 16 joints
Links:
- link base_link: geometry visual box size=3.9425 3.5385 1.904
- link left_arm1: geometry visual box size=1.725 1.402 1.9545
- link left_arm2: geometry visual box size=1.29 2.1 1.45
- link left_arm3: geometry visual box size=1.84 2.615 1
- link left_arm4: geometry visual box size=1.26 1.67 1.45
- link left_leg1: geometry visual box size=1.774 1.095 3.31
- link left_leg2: geometry visual box size=4.77 1.279 .973
- link left_leg3: geometry visual box size=4.388 1.316 1.076
- link left_leg4: geometry visual box size=1.67 1.96 1.346
- link right_arm1: geometry visual box size=1.725 -1.402 1.9545
- link right_arm2: geometry visual box size=1.29 -2.1 1.45
- link right_arm3: geometry visual box size=1.84 -2.615 1
- link right_arm4: geometry visual box size=1.26 -1.67 1.45
- link right_leg1: geometry visual box size=1.774 1.095 3.31
- link right_leg2: geometry visual box size=4.77 1.279 .973
- link right_leg3: geometry visual box size=4.388 1.316 1.076
- link right_leg4: geometry visual box size=1.67 1.96 1.346
Joints:
- joint [ARM] left1_to_left2 : limit lower=-3.14 upper=3.14 effort=1000 velocity=0.5 -> lower=-1.57 upper=1.57 effort=1000 velocity=0.5; origin xyz=0 .6 0 -> xyz=0 1.402 0
- joint [ARM] left2_to_left3 : origin xyz=0 .6 0 -> xyz=0 2.1 0
- joint [ARM] left3_to_left4 : limit lower=-3.14 upper=3.14 effort=1000 velocity=0.5 -> lower=-1.57 upper=1.57 effort=1000 velocity=0.5; origin xyz=0 .6 0 -> xyz=0 2.615 0
- joint [ARM] right1_to_right2: axis 0 0 1 -> 0 0 1 ; limit lower=-3.14 upper=3.14 effort=1000 velocity=0.5 -> lower=-1.57 upper=1.57 effort=1000 velocity=0.5; origin xyz=0 -.6 0 -> xyz=0 -1.402 0
- joint [ARM] right2_to_right3: origin xyz=0 -.6 0 -> xyz=0 -2.1 0
- joint [ARM] right3_to_right4: limit lower=-3.14 upper=3.14 effort=1000 velocity=0.5 -> lower=-1.57 upper=1.57 effort=1000 velocity=0.5; origin xyz=0 -.6 0 -> xyz=0 -2.615 0
- joint [LEG] left1_to_left2: limit lower=-3.14 upper=3.14 effort=1000 velocity=0.5 -> lower=0 upper=1.57 effort=1000 velocity=0.5; origin xyz=.6 0 0 -> xyz=1.774 0 0
- joint [LEG] left2_to__left3: limit lower=-3.14 upper=3.14 effort=1000 velocity=0.5 -> lower=0 upper=1.57 effort=1000 velocity=0.5; origin xyz=.6 0 0 -> xyz=4.77 0 0
- joint [LEG] left3_to_left4: limit lower=-3.14 upper=3.14 effort=1000 velocity=0.5 -> lower=-1.57 upper=1.57 effort=1000 velocity=0.5; origin xyz=.6 0 0 -> xyz=4.388 0 0
- joint [LEG] right1_to_right2: limit lower=-3.14 upper=3.14 effort=1000 velocity=0.5 -> lower=0 upper=1.57 effort=1000 velocity=0.5; origin xyz=0.6 0 0 -> xyz=1.774 0 0
- joint [LEG] right3_to_right4: limit lower=-3.14 upper=3.14 effort=1000 velocity=0.5 -> lower=-1.57 upper=1.57 effort=1000 velocity=0.5; origin xyz=0.6 0 0 -> xyz=4.388 0 0
- joint base_to_left_arm: origin xyz=-.85 .75 0 -> xyz=-1.10875 1.76925  0
- joint base_to_left_leg: limit lower=-3.14 upper=3.14 effort=1000 velocity=0.5 -> lower=-1.05 upper=1.05 effort=1000 velocity=0.5; origin xyz=1 .6 0 -> xyz=1.97125 1.22175  0
- joint base_to_right_arm: origin xyz=-.85 -.75 0 -> xyz=-1.10875 -1.76925  0
- joint base_to_right_leg: limit lower=-3.14 upper=3.14 effort=1000 velocity=0.5 -> lower=-1.05 upper=1.05 effort=1000 velocity=0.5; origin xyz=1 -.6 0 -> xyz=1.97125 -1.22175  0
- joint right2_to_right3: limit lower=-3.14 upper=3.14 effort=1000 velocity=0.5 -> lower=0 upper=1.57 effort=1000 velocity=0.5; origin xyz=0.6 0 0 -> xyz=4.77 0 0
